File: mcu.sch (KiCad schematic (older format))
At the start: 32 parts, among them J10 USB_C_Receptacle_USB2.0, J4 debug, J5 Conn_01x16_Male, J6 Conn_01x16_Male, U3 STM32F407VETx, Y1 12Mhz

Commit message: Various fixes
Parts:
- added R16, R17: 10k, symbol Device:R
- added SW1, SW2: SW_MEC_5E, symbol Switch:SW_MEC_5E
- R10, R8, R9: value 75 -> 120
- R7: value 75 -> 120; footprint (none) -> 120
- gave numbers to parts that had none: 3
Connections:
- net 3.3V: now also SW1.3 (K), SW1.4 (A), SW2.3 (K), SW2.4 (A)
- net GND: now also R16.2, R17.2; no longer U3.94 (BOOT0)
- net NRST: now reaches U3.14 (NRST)
- net NRST: now also R16.1, SW2.1, SW2.2
- new net BOOT0: R17.1, SW1.1, SW1.2, U3.94 (BOOT0)
Changed lines of the file:
@@
 L power:GND #PWR018
 U 1 1 6007ECDF
-P 1450 1600
-F 0 "#PWR018" H 1450 1350 50  0001 C CNN
-F 1 "GND" H 1455 1427 50  0000 C CNN
-F 2 "" H 1450 1600 50  0001 C CNN
-F 3 "" H 1450 1600 50  0001 C CNN
-	1    1450 1600
-	1    0    0    -1
-$EndComp
-Wire Wire Line
-	1450 1600 2100 1600
+P 1300 2100
+F 0 "#PWR018" H 1300 1850 50  0001 C CNN
+F 1 "GND" H 1305 1927 50  0000 C CNN
+F 2 "" H 1300 2100 50  0001 C CNN
+F 3 "" H 1300 2100 50  0001 C CNN
+	1    1300 2100
+	1    0    0    -1
+$EndComp
 $Comp
 L Device:Crystal Y1
@@
 P 10000 3950
 F 0 "R7" V 9793 3950 50  0000 C CNN
-F 1 "75" V 9884 3950 50  0000 C CNN
-F 2 "" V 9930 3950 50  0001 C CNN
+F 1 "120" V 9884 3950 50  0000 C CNN
+F 2 "120" V 9930 3950 50  0001 C CNN
 F 3 "~" H 10000 3950 50  0001 C CNN
 	1    10000 3950
@@
 P 10050 4600
 F 0 "R8" V 9843 4600 50  0000 C CNN
-F 1 "75" V 9934 4600 50  0000 C CNN
+F 1 "120" V 9934 4600 50  0000 C CNN
 F 2 "" V 9980 4600 50  0001 C CNN
 F 3 "~" H 10050 4600 50  0001 C CNN
@@
 P 10050 5250
 F 0 "R9" V 9843 5250 50  0000 C CNN
-F 1 "75" V 9934 5250 50  0000 C CNN
+F 1 "120" V 9934 5250 50  0000 C CNN
 F 2 "" V 9980 5250 50  0001 C CNN
 F 3 "~" H 10050 5250 50  0001 C CNN
@@
 P 10050 5900
 F 0 "R10" V 9843 5900 50  0000 C CNN
-F 1 "75" V 9934 5900 50  0000 C CNN
+F 1 "120" V 9934 5900 50  0000 C CNN
 F 2 "" V 9980 5900 50  0001 C CNN
 F 3 "~" H 10050 5900 50  0001 C CNN
@@
 	8300 3750 8500 3750
 $Comp
-L Device:R R?
+L Device:R R11
 U 1 1 601DC33F
 P 7550 4450
-F 0 "R?" H 7620 4496 50  0000 L CNN
+F 0 "R11" H 7620 4496 50  0000 L CNN
 F 1 "5.1k" H 7620 4405 50  0000 L CNN
 F 2 "" V 7480 4450 50  0001 C CNN
@@
 $EndComp
 $Comp
-L Device:R R?
+L Device:R R12
 U 1 1 601DC805
 P 7900 4450
-F 0 "R?" H 7970 4496 50  0000 L CNN
+F 0 "R12" H 7970 4496 50  0000 L CNN
 F 1 "5.1k" H 7970 4405 50  0000 L CNN
 F 2 "" V 7830 4450 50  0001 C CNN
@@
 	7900 4150 7900 4300
 $Comp
-L power:GND #PWR?
+L power:GND #PWR028
 U 1 1 601F11CD
 P 7550 4700
-F 0 "#PWR?" H 7550 4450 50  0001 C CNN
+F 0 "#PWR028" H 7550 4450 50  0001 C CNN
 F 1 "GND" H 7555 4527 50  0000 C CNN
 F 2 "" H 7550 4700 50  0001 C CNN
@@
 	7550 4700 7550 4600
 $Comp
-L power:GND #PWR?
+L power:GND #PWR029
 U 1 1 601FB749
 P 7900 4700
-F 0 "#PWR?" H 7900 4450 50  0001 C CNN
+F 0 "#PWR029" H 7900 4450 50  0001 C CNN
 F 1 "GND" H 7905 4527 50  0000 C CNN
 F 2 "" H 7900 4700 50  0001 C CNN
@@
 	7900 4700 7900 4600
 $Comp
-L Device:R R?
+L Device:R R13
 U 1 1 60234B64
 P 8300 4450
-F 0 "R?" H 8370 4496 50  0000 L CNN
+F 0 "R13" H 8370 4496 50  0000 L CNN
 F 1 "1M" H 8370 4405 50  0000 L CNN
 F 2 "" V 8230 4450 50  0001 C CNN
@@
 $EndComp
 $Comp
-L power:GND #PWR?
+L power:GND #PWR030
 U 1 1 6023573F
 P 8300 4700
-F 0 "#PWR?" H 8300 4450 50  0001 C CNN
+F 0 "#PWR030" H 8300 4450 50  0001 C CNN
 F 1 "GND" H 8305 4527 50  0000 C CNN
 F 2 "" H 8300 4700 50  0001 C CNN
@@
 Wire Wire Line
 	6750 3950 8300 3950
+$Comp
+L Switch:SW_MEC_5E SW1
+U 1 1 602AEEE9
+P 7950 5700
+F 0 "SW1" H 7950 6085 50  0000 C CNN
+F 1 "SW_MEC_5E" H 7950 5994 50  0000 C CNN
+F 2 "" H 7950 6000 50  0001 C CNN
+F 3 "http://www.apem.com/int/index.php?controller=attachment&id_attachment=1371" H 7950 6000 50  0001 C CNN
+	1    7950 5700
+	1    0    0    -1
+$EndComp
+$Comp
+L Switch:SW_MEC_5E SW2
+U 1 1 602B029E
+P 7950 6250
+F 0 "SW2" H 7950 6635 50  0000 C CNN
+F 1 "SW_MEC_5E" H 7950 6544 50  0000 C CNN
+F 2 "" H 7950 6550 50  0001 C CNN
+F 3 "http://www.apem.com/int/index.php?controller=attachment&id_attachment=1371" H 7950 6550 50  0001 C CNN
+	1    7950 6250
+	1    0    0    -1
+$EndComp
+$Comp
+L Device:R R17
+U 1 1 602B1BCD
+P 1300 1900
+F 0 "R17" H 1370 1946 50  0000 L CNN
+F 1 "10k" H 1370 1855 50  0000 L CNN
+F 2 "" V 1230 1900 50  0001 C CNN
+F 3 "~" H 1300 1900 50  0001 C CNN
+	1    1300 1900
+	1    0    0    -1
+$EndComp
+Wire Wire Line
+	1300 2050 1300 2100
+Wire Wire Line
+	1300 1600 1300 1750
+Text Label 1300 1600 2    50   ~ 0
+BOOT0
+Wire Wire Line
+	7750 5600 7700 5600
+Wire Wire Line
+	7700 5600 7700 5650
+Wire Wire Line
+	7700 5700 7750 5700
+Text Label 7600 5650 2    50   ~ 0
+BOOT0
+Wire Wire Line
+	7600 5650 7700 5650
+Connection ~ 7700 5650
+Wire Wire Line
+	7700 5650 7700 5700
+Text GLabel 8250 5650 2    50   Input ~ 0
+3.3V
+Wire Wire Line
+	8150 5600 8200 5600
+Wire Wire Line
+	8200 5600 8200 5650
+Wire Wire Line
+	8200 5700 8150 5700
+Wire Wire Line
+	8250 5650 8200 5650
+Connection ~ 8200 5650
+Wire Wire Line
+	8200 5650 8200 5700
+Wire Wire Line
+	1300 1600 2100 1600
+$Comp
+L power:GND #PWR031
+U 1 1 60338445
+P 750 2100
+F 0 "#PWR031" H 750 1850 50  0001 C CNN
+F 1 "GND" H 755 1927 50  0000 C CNN
+F 2 "" H 750 2100 50  0001 C CNN
+F 3 "" H 750 2100 50  0001 C CNN
+	1    750  2100
+	1    0    0    -1
+$EndComp
+$Comp
+L Device:R R16
+U 1 1 6033844B
+P 750 1900
+F 0 "R16" H 820 1946 50  0000 L CNN
+F 1 "10k" H 820 1855 50  0000 L CNN
+F 2 "" V 680 1900 50  0001 C CNN
+F 3 "~" H 750 1900 50  0001 C CNN
+	1    750  1900
+	1    0    0    -1
+$EndComp
+Wire Wire Line
+	750  2050 750  2100
+Wire Wire Line
+	750  1750 750  1400
+Wire Wire Line
+	750  1400 2100 1400
+Text Label 750  1400 2    50   ~ 0
+NRST
+Text Label 7600 6200 2    50   ~ 0
+NRST
+Wire Wire Line
+	7600 6200 7700 6200
+Wire Wire Line
+	7700 6200 7700 6150
+Wire Wire Line
+	7700 6150 7750 6150
+Wire Wire Line
+	7700 6200 7700 6250
+Wire Wire Line
+	7700 6250 7750 6250
+Connection ~ 7700 6200
+Text GLabel 8250 6200 2    50   Input ~ 0
+3.3V
+Wire Wire Line
+	8150 6150 8200 6150
+Wire Wire Line
+	8200 6150 8200 6200
+Wire Wire Line
+	8200 6250 8150 6250
+Wire Wire Line
+	8250 6200 8200 6200
+Connection ~ 8200 6200
+Wire Wire Line
+	8200 6200 8200 6250
 $EndSCHEMATC
