File: mcu.sch (KiCad schematic (older format))
At the start: 34 parts, among them J10 DX07S016JA1R1500, J11 Conn_02x08_Odd_Even, J7 digital, J8 analog, J9 debug, U3 ATSAME51J18A-A, Y1 8Mhz

Commit message: "0.1u" -> "100n"; use 1206 10u for bulk decoupling
The 1206 size has a much better derating-vs-bias-voltage curve.
Parts:
- C12, C15, C6, C8: footprint Capacitor_SMD:C_0603_1608Metric -> Capacitor_SMD:C_1206_3216Metric
Changed lines of the file:
@@
 F 0 "C8" H 5465 3396 50  0000 L CNN
 F 1 "10u" H 5465 3305 50  0000 L CNN
-F 2 "Capacitor_SMD:C_0603_1608Metric" H 5388 3200 50  0001 C CNN
+F 2 "Capacitor_SMD:C_1206_3216Metric" H 5388 3200 50  0001 C CNN
 F 3 "~" H 5350 3350 50  0001 C CNN
 	1    5350 3350
@@
 F 0 "C12" H 5915 3396 50  0000 L CNN
 F 1 "10u" H 5915 3305 50  0000 L CNN
-F 2 "Capacitor_SMD:C_0603_1608Metric" H 5838 3200 50  0001 C CNN
+F 2 "Capacitor_SMD:C_1206_3216Metric" H 5838 3200 50  0001 C CNN
 F 3 "~" H 5800 3350 50  0001 C CNN
 	1    5800 3350
@@
 F 0 "C15" H 6365 3396 50  0000 L CNN
 F 1 "10u" H 6365 3305 50  0000 L CNN
-F 2 "Capacitor_SMD:C_0603_1608Metric" H 6288 3200 50  0001 C CNN
+F 2 "Capacitor_SMD:C_1206_3216Metric" H 6288 3200 50  0001 C CNN
 F 3 "~" H 6250 3350 50  0001 C CNN
 	1    6250 3350
@@
 F 0 "C6" H 2015 796 50  0000 L CNN
 F 1 "10u" H 2015 705 50  0000 L CNN
-F 2 "Capacitor_SMD:C_0603_1608Metric" H 1938 600 50  0001 C CNN
+F 2 "Capacitor_SMD:C_1206_3216Metric" H 1938 600 50  0001 C CNN
 F 3 "~" H 1900 750 50  0001 C CNN
 	1    1900 750
