File: TI_Codec.sch (KiCad schematic (older format))
At the start: 11 parts, among them U5 TLV320AIC3105IRHBR

Commit message: Swap TI codec footprint for builtin QFN
5x5mm size, 0.5mm pitch, 3.45mm exposed pad.  TI recommends the thermal
vias, though on something this low-power, I think that's overkill.

I had to use a copper-fill keepout and manually draw traces to keep the
pads from being horribly misshaped.
Parts:
- U5: footprint TLV320AIC3105:TLV320AIC3105IRHBR -> Package_DFN_QFN:QFN-32-1EP_5x5mm_P0.5mm_EP3.45x3.45mm_ThermalVias
Changed lines of the file:
@@
 F 0 "U5" H 3950 2537 60  0000 C CNN
 F 1 "TLV320AIC3105IRHBR" H 3950 2431 60  0000 C CNN
-F 2 "TLV320AIC3105:TLV320AIC3105IRHBR" H 3950 2390 60  0001 C CNN
+F 2 "Package_DFN_QFN:QFN-32-1EP_5x5mm_P0.5mm_EP3.45x3.45mm_ThermalVias" H 3950 2390 60  0001 C CNN
 F 3 "" H 2350 2150 60  0000 C CNN
 	1    2350 2150
@@
 F 0 "U5" H 8828 1553 60  0000 L CNN
 F 1 "TLV320AIC3105IRHBR" H 8828 1447 60  0000 L CNN
-F 2 "TLV320AIC3105:TLV320AIC3105IRHBR" H 9100 2390 60  0001 C CNN
+F 2 "Package_DFN_QFN:QFN-32-1EP_5x5mm_P0.5mm_EP3.45x3.45mm_ThermalVias" H 9100 2390 60  0001 C CNN
 F 3 "" H 7500 2150 60  0000 C CNN
 	2    7500 2150
